File: novo_projeto/novo_projeto.kicad_sch (KiCad schematic)
At the start: 6 parts, among them SW1 SW_DPST, U1 LCD_16X2, U2 LCD_16X2

Commit message: bluepill add
Parts:
- added U3: Bluepill, symbol Clemonini_Lbrary:Bluepill
Changed lines of the file:
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@@
+		)
+	)
+	(symbol
+		(lib_id "Clemonini_Lbrary:Bluepill")
+		(at 20.32 33.02 0)
+		(unit 1)
+		(exclude_from_sim no)
+		(in_bom yes)
+		(on_board yes)
+		(dnp no)
+		(fields_autoplaced yes)
+		(property "Reference" "U3"
+			(at 34.29 27.94 0)
+			(effects
+				(font
+					(size 1.27 1.27)
+				)
+			)
+		)
+		(property "Value" "Bluepill"
+			(at 34.29 30.48 0)
+			(effects
+				(font
+					(size 1.27 1.27)
+				)
+			)
+		)
+		(property "Footprint" ""
+			(at 12.7 33.02 0)
+			(effects
+				(font
+					(size 1.27 1.27)
+				)
+				(hide yes)
+			)
+		)
+		(property "Datasheet" ""
+			(at 12.7 33.02 0)
+			(effects
+				(font
+					(size 1.27 1.27)
+				)
+				(hide yes)
+			)
+		)
+		(property "Description" ""
+			(at 76.708 76.2 0)
+			(effects
+				(font
+					(size 1.27 1.27)
+				)
+				(hide yes)
+			)
+		)
+		(pin "12"
+		)
+		(pin "10"
+		)
+		(pin "1"
+		)
+		(pin "13"
+		)
+		(pin "17"
+		)
+		(pin "15"
+		)
+		(pin "11"
+		)
+		(pin "16"
+		)
+		(pin "14"
+		)
+		(pin "18"
+		)
+		(pin "19"
+		)
+		(pin "2"
+		)
+		(pin "20"
+		)
+		(pin "21"
+		)
+		(pin "22"
+		)
+		(pin "23"
+		)
+		(pin "24"
+		)
+		(pin "25"
+		)
+		(pin "26"
+		)
+		(pin "27"
+		)
+		(pin "28"
+		)
+		(pin "29"
+		)
+		(pin "3"
+		)
+		(pin "30"
+		)
+		(pin "31"
+		)
+		(pin "32"
+		)
+		(pin "33"
+		)
+		(pin "34"
+		)
+		(pin "35"
+		)
+		(pin "36"
+		)
+		(pin "37"
+		)
+		(pin "38"
+		)
+		(pin "39"
+		)
+		(pin "4"
+		)
+		(pin "40"
+		)
+		(pin "5"
+		)
+		(pin "6"
+		)
+		(pin "7"
+		)
+		(pin "8"
+		)
+		(pin "9"
+		)
+		(instances
+			(project ""
+				(path "/c0ea3d43-a3f7-4350-879c-bb04e86ffdf1"
+					(reference "U3")
+					(unit 1)
+				)
+			)
 		)
 	)

Commit message: template config
Other:
- company: (none) -> Pedro Clemonini
- title: (none) -> Aula LPE06
Changed lines of the file:
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@@
 	(generator_version "8.0")
 	(paper "A4")
+	(title_block
+		(title "Aula LPE06")
+		(rev "1")
+		(company "Pedro Clemonini")
+		(comment 1 "Projeto teste")
+	)
 	(junction
 		(at 78.74 73.66)
